Commit message: chore(samples): add basic OBJ link meshes and reference in sample URDF; playback UI wiring complete

File: apps/web/public/robots/sample-arm-01/urdf/sample.urdf (robot description, URDF)
Before this commit: robot sample-arm-01, 2 links, 1 joints
Links:
- link base: geometry visual mesh filename=/robots/sample-arm-01/links/base.obj
- link link1: geometry visual mesh filename=/robots/sample-arm-01/links/link1.obj

Commit message: more elaborate rendering

File: apps/web/public/robots/sample-arm-01/urdf/sample.urdf (robot description, URDF)
Before this commit: robot sample-arm-01, 2 links, 1 joints
Links:
- added link link2; visual box size=0.18 0.6 0.18
- link base: geometry visual mesh filename=../links/base.obj
- link link1: geometry visual mesh filename=../links/link1.obj
Joints:
- added joint joint2: type revolute, parent link1, child link2, origin xyz=0 0.4 0 rpy=0 0 0, axis 0 1 0, limit lower=-1.2 upper=1.2 velocity=1

Commit message: enhanced simulation

File: apps/web/public/robots/sample-arm-01/urdf/sample.urdf (robot description, URDF)
Before this commit: robot sample-arm-01, 3 links, 2 joints
Links:
- link base: geometry visual mesh filename=../links/base.glb
- link link1: geometry visual mesh filename=../links/link1.glb
